File: _pcb/VestibularVR H1-module v1.0/VestibularVR H1-module v1.0.brd (EAGLE design)
At the start: 43 x 57.4 mm, 67 parts, among them IC1 FT232RL, IC2 74LVC1G07DBV, IC3 LP5907MFX-3.3, IC4 74LVC1G07DBV, IC5 74LVC1G07DBV, IC6 74LVC1G07DBV, IC7 USBLC6-2SC6, IC8 ATXMEGA32A4U, T1 DMG1012UW, T2 DMG1012UW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

Commit message: VestibularVR H1BOM updates & Lick Sensor step on
- VestibularVR H1
. component ref updated
. BOM file updated

- Lick Sensor module v1.0
. still only on schematic design
Parts:
- IC2, IC4, IC5, IC6: value 74LVC1G07DBV -> 74VHC1GT126DT1G
Changed lines of the file:
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@@
 <attribute name="VALUE" x="28.4882" y="36.4132" size="1.27" layer="27" ratio="10" rot="R90"/>
 </element>
-<element name="IC2" library="VestibularVR H1-module v1.0" package="SOT23-5" package3d_urn="urn:adsk.eagle:package:2406/2" value="74LVC1G07DBV" x="10.675" y="42.436" smashed="yes" rot="MR270">
+<element name="IC2" library="VestibularVR H1-module v1.0" package="SOT23-5" package3d_urn="urn:adsk.eagle:package:2406/2" value="74VHC1GT126DT1G" x="10.675" y="42.436" smashed="yes" rot="MR270">
 <attribute name="MPN" value="M74VHC1GT126DT1G" x="10.675" y="42.436" size="1.778" layer="28" rot="MR270" display="off"/>
 <attribute name="NAME" x="9.682" y="40.7232" size="0.8128" layer="26" font="vector" ratio="15" rot="MR180"/>
@@
 <attribute name="VALUE" x="14.485" y="44.976" size="1.27" layer="28" rot="MR270"/>
 </element>
-<element name="IC4" library="VestibularVR H1-module v1.0" package="SOT23-5" package3d_urn="urn:adsk.eagle:package:2406/2" value="74LVC1G07DBV" x="10.675" y="51.072" smashed="yes" rot="MR270">
+<element name="IC4" library="VestibularVR H1-module v1.0" package="SOT23-5" package3d_urn="urn:adsk.eagle:package:2406/2" value="74VHC1GT126DT1G" x="10.675" y="51.072" smashed="yes" rot="MR270">
 <attribute name="MPN" value="M74VHC1GT126DT1G" x="10.675" y="51.072" size="1.778" layer="28" rot="MR270" display="off"/>
 <attribute name="NAME" x="9.6072" y="49.4124" size="0.8128" layer="26" font="vector" ratio="15" rot="MR180"/>
@@
 <attribute name="VALUE" x="14.485" y="53.612" size="1.27" layer="28" rot="MR270"/>
 </element>
-<element name="IC5" library="VestibularVR H1-module v1.0" package="SOT23-5" package3d_urn="urn:adsk.eagle:package:2406/2" value="74LVC1G07DBV" x="12.5566" y="24.3972" smashed="yes" rot="MR90">
+<element name="IC5" library="VestibularVR H1-module v1.0" package="SOT23-5" package3d_urn="urn:adsk.eagle:package:2406/2" value="74VHC1GT126DT1G" x="12.5566" y="24.3972" smashed="yes" rot="MR90">
 <attribute name="MPN" value="M74VHC1GT126DT1G" x="12.5566" y="24.3972" size="1.778" layer="28" rot="MR90" display="off"/>
 <attribute name="NAME" x="11.7034" y="26.996" size="0.8128" layer="26" font="vector" ratio="15" rot="MR180"/>
@@
 <attribute name="VALUE" x="8.7466" y="21.8572" size="1.27" layer="28" rot="MR90"/>
 </element>
-<element name="IC6" library="VestibularVR H1-module v1.0" package="SOT23-5" package3d_urn="urn:adsk.eagle:package:2406/2" value="74LVC1G07DBV" x="12.5566" y="35.2374" smashed="yes" rot="MR90">
+<element name="IC6" library="VestibularVR H1-module v1.0" package="SOT23-5" package3d_urn="urn:adsk.eagle:package:2406/2" value="74VHC1GT126DT1G" x="12.5566" y="35.2374" smashed="yes" rot="MR90">
 <attribute name="MPN" value="M74VHC1GT126DT1G" x="12.5566" y="35.2374" size="1.778" layer="28" rot="MR90" display="off"/>
 <attribute name="NAME" x="11.4542" y="33.2608" size="0.8128" layer="26" font="vector" ratio="15" rot="MR180"/>

Commit message: >> VestibularVR H1-module v1.0: corrected part numbers
>> VestibularVR H1-module v1.0
- notes added on schematic
	. buffers with wrong pn - corrected OEPS code; still wrong buffers' symbol
	generated new BOM with corrected pn
Parts:
- IC2, IC4, IC5, IC6: value 74VHC1GT126DT1G -> SN74LVC1G125DBVT
Changed lines of the file:
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@@
 <attribute name="VALUE" x="28.4882" y="36.4132" size="1.27" layer="27" ratio="10" rot="R90"/>
 </element>
-<element name="IC2" library="VestibularVR H1-module v1.0" package="SOT23-5" package3d_urn="urn:adsk.eagle:package:2406/2" value="74VHC1GT126DT1G" x="10.675" y="42.436" smashed="yes" rot="MR270">
-<attribute name="MPN" value="M74VHC1GT126DT1G" x="10.675" y="42.436" size="1.778" layer="28" rot="MR270" display="off"/>
+<element name="IC2" library="VestibularVR H1-module v1.0" package="SOT23-5" package3d_urn="urn:adsk.eagle:package:2406/2" value="SN74LVC1G125DBVT" x="10.675" y="42.436" smashed="yes" rot="MR270">
+<attribute name="MPN" value="SN74LVC1G125DBVT" x="10.675" y="42.436" size="1.778" layer="28" rot="MR270" display="off"/>
 <attribute name="NAME" x="9.682" y="40.7232" size="0.8128" layer="26" font="vector" ratio="15" rot="MR180"/>
-<attribute name="OEPS" value="OEPS080017" x="10.675" y="42.436" size="1.778" layer="28" rot="MR270" display="off"/>
+<attribute name="OEPS" value="OEPS080029" x="10.675" y="42.436" size="1.778" layer="28" rot="MR270" display="off"/>
 <attribute name="VALUE" x="14.485" y="44.976" size="1.27" layer="28" rot="MR270"/>
 </element>
-<element name="IC4" library="VestibularVR H1-module v1.0" package="SOT23-5" package3d_urn="urn:adsk.eagle:package:2406/2" value="74VHC1GT126DT1G" x="10.675" y="51.072" smashed="yes" rot="MR270">
-<attribute name="MPN" value="M74VHC1GT126DT1G" x="10.675" y="51.072" size="1.778" layer="28" rot="MR270" display="off"/>
+<element name="IC4" library="VestibularVR H1-module v1.0" package="SOT23-5" package3d_urn="urn:adsk.eagle:package:2406/2" value="SN74LVC1G125DBVT" x="10.675" y="51.072" smashed="yes" rot="MR270">
+<attribute name="MPN" value="SN74LVC1G125DBVT" x="10.675" y="51.072" size="1.778" layer="28" rot="MR270" display="off"/>
 <attribute name="NAME" x="9.6072" y="49.4124" size="0.8128" layer="26" font="vector" ratio="15" rot="MR180"/>
-<attribute name="OEPS" value="OEPS080017" x="10.675" y="51.072" size="1.778" layer="28" rot="MR270" display="off"/>
+<attribute name="OEPS" value="OEPS080029" x="10.675" y="51.072" size="1.778" layer="28" rot="MR270" display="off"/>
 <attribute name="VALUE" x="14.485" y="53.612" size="1.27" layer="28" rot="MR270"/>
 </element>
-<element name="IC5" library="VestibularVR H1-module v1.0" package="SOT23-5" package3d_urn="urn:adsk.eagle:package:2406/2" value="74VHC1GT126DT1G" x="12.5566" y="24.3972" smashed="yes" rot="MR90">
-<attribute name="MPN" value="M74VHC1GT126DT1G" x="12.5566" y="24.3972" size="1.778" layer="28" rot="MR90" display="off"/>
+<element name="IC5" library="VestibularVR H1-module v1.0" package="SOT23-5" package3d_urn="urn:adsk.eagle:package:2406/2" value="SN74LVC1G125DBVT" x="12.5566" y="24.3972" smashed="yes" rot="MR90">
+<attribute name="MPN" value="SN74LVC1G125DBVT" x="12.5566" y="24.3972" size="1.778" layer="28" rot="MR90" display="off"/>
 <attribute name="NAME" x="11.7034" y="26.996" size="0.8128" layer="26" font="vector" ratio="15" rot="MR180"/>
-<attribute name="OEPS" value="OEPS080017" x="12.5566" y="24.3972" size="1.778" layer="28" rot="MR90" display="off"/>
+<attribute name="OEPS" value="OEPS080029" x="12.5566" y="24.3972" size="1.778" layer="28" rot="MR90" display="off"/>
 <attribute name="VALUE" x="8.7466" y="21.8572" size="1.27" layer="28" rot="MR90"/>
 </element>
-<element name="IC6" library="VestibularVR H1-module v1.0" package="SOT23-5" package3d_urn="urn:adsk.eagle:package:2406/2" value="74VHC1GT126DT1G" x="12.5566" y="35.2374" smashed="yes" rot="MR90">
-<attribute name="MPN" value="M74VHC1GT126DT1G" x="12.5566" y="35.2374" size="1.778" layer="28" rot="MR90" display="off"/>
+<element name="IC6" library="VestibularVR H1-module v1.0" package="SOT23-5" package3d_urn="urn:adsk.eagle:package:2406/2" value="SN74LVC1G125DBVT" x="12.5566" y="35.2374" smashed="yes" rot="MR90">
+<attribute name="MPN" value="SN74LVC1G125DBVT" x="12.5566" y="35.2374" size="1.778" layer="28" rot="MR90" display="off"/>
 <attribute name="NAME" x="11.4542" y="33.2608" size="0.8128" layer="26" font="vector" ratio="15" rot="MR180"/>
-<attribute name="OEPS" value="OEPS080017" x="12.5566" y="35.2374" size="1.778" layer="28" rot="MR90" display="off"/>
+<attribute name="OEPS" value="OEPS080029" x="12.5566" y="35.2374" size="1.778" layer="28" rot="MR90" display="off"/>
 <attribute name="VALUE" x="8.7466" y="32.6974" size="1.27" layer="28" rot="MR90"/>
 </element>
@@
 <attribute name="MPN" value="04025A470JAT2A" x="35.726" y="47.355" size="1.778" layer="27" rot="R270" display="off"/>
 <attribute name="NAME" x="24.1878" y="46.5488" size="0.8128" layer="25" font="vector" ratio="15" rot="R90"/>
-<attribute name="OEPS" value="OEPS080013" x="22.726" y="47.355" size="1.778" layer="27" rot="R270" display="off"/>
+<attribute name="OEPS" value="n.a." x="22.726" y="47.355" size="1.778" layer="27" rot="R270" display="off"/>
 <attribute name="VALUE" x="20.821" y="47.99" size="1.27" layer="27" rot="R270"/>
 </element>
@@
 <attribute name="MPN" value="04025A470JAT2A" x="14.726" y="47.348" size="1.778" layer="27" rot="R90" display="off"/>
 <attribute name="NAME" x="23.4004" y="53.6288" size="0.8128" layer="25" font="vector" ratio="15" rot="R270"/>
-<attribute name="OEPS" value="OEPS080013" x="22.726" y="52.848" size="1.778" layer="27" rot="R90" display="off"/>
+<attribute name="OEPS" value="n.a." x="22.726" y="52.848" size="1.778" layer="27" rot="R90" display="off"/>
 <attribute name="VALUE" x="24.631" y="52.213" size="1.27" layer="27" rot="R90"/>
 </element>
@@
 <attribute name="MPN" value="04025A470JAT2A" x="24.34715" y="32.4612" size="1.778" layer="27" rot="R180" display="off"/>
 <attribute name="NAME" x="23.07715" y="33.655" size="0.8128" layer="25" font="vector" ratio="15" rot="R180"/>
-<attribute name="OEPS" value="OEPS080013" x="24.34715" y="32.4612" size="1.778" layer="27" rot="R180" display="off"/>
+<attribute name="OEPS" value="n.a." x="24.34715" y="32.4612" size="1.778" layer="27" rot="R180" display="off"/>
 <attribute name="VALUE" x="24.98215" y="34.3662" size="1.27" layer="27" rot="R180"/>
 </element>
@@
 </element>
 <element name="X1" library="con-samtec" library_urn="urn:adsk.eagle:library:184" package="TSW-105-02-S-D" value="2x5 header" x="25.908" y="8.382" smashed="yes" rot="R90">
-<attribute name="MF" value="" x="25.908" y="8.382" size="1.778" layer="27" rot="R90" display="off"/>
-<attribute name="MPN" value="2x5 header" x="25.908" y="8.382" size="1.778" layer="27" rot="R90" display="off"/>
 <attribute name="NAME" x="25.6032" y="15.113" size="0.8128" layer="25" font="vector" ratio="15"/>
 <attribute name="OC_FARNELL" value="unknown" x="25.908" y="8.382" size="1.778" layer="27" rot="R90" display="off"/>
