File: Hardware/PCB/VestibularH1.brd (EAGLE design)
At the start: 43 x 57.4 mm, 67 parts, among them IC1 FT232RL, IC2 SN74LVC1G125DBVT, IC3 LP5907MFX-3.3, IC4 SN74LVC1G125DBVT, IC5 SN74LVC1G125DBVT, IC6 SN74LVC1G125DBVT, IC7 USBLC6-2SC6, IC8 ATXMEGA32A4U, T1 DMG1012UW, T2 DMG1012UW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

Commit message: Replaced files with version 1.1.
Parts:
- removed IC6: SN74LVC1G125DBVT, VestibularVR H1-module v1.0:SOT23-5
- added IC9: M74VHC1GT126DT1G, VestibularVR H1-module v1.0:TSOP-5
- C10: device rcl:C0603K -> rcl:C0603
- IC2, IC4, IC5: value SN74LVC1G125DBVT -> M74VHC1GT126DT1G; device VestibularVR H1-module v1.0:SOT23-5 -> VestibularVR H1-module v1.0:TSOP-5
- moved IC5 26.8 mm to (9.65, 51.1), turned to 270 degrees
- moved IC4 8.97 mm to (9.65, 42.2)
- moved IC2 7.29 mm to (12.2, 35.3), turned to 90 degrees
- moved C6 5.67 mm to (23.5, 47.2), turned to 270 degrees
- moved C4 3.42 mm to (23.5, 50.7), turned to 90 degrees
- moved C13 0.51 mm to (23.8, 32.5)
- renumbered REWARD_VALVES to VALVES
Connections:
- net +3V3: now also IC2.1, IC2.5, IC9.1, IC9.5; no longer IC5.5, IC6.5
- net +3V3_U: now also SV2.2; no longer SV2.6
- net GND: now also IC9.3, SV2.6; no longer IC6.3, SV2.2
- net LICK_PORT_1: now also IC2.2; no longer IC6.2
- net LICK_PORT_2: now also IC9.2; no longer IC5.2
- net N$14: now also IC4.1, IC4.5; no longer IC2.5
- net N$4: now also IC4.4; no longer IC2.4
- net N$5: now also IC5.1, IC5.5; no longer IC4.5
- net N$8: now also IC5.4; no longer IC4.4
- net PDI_CLK: now also SV2.5; no longer SV2.1
- net PDI_DATA: now also SV2.1; no longer SV2.5
- net USBDM: now also IC7.P$3; no longer IC7.P$1
- net USBDP: now also IC7.P$1; no longer IC7.P$3
- net U_CAM1_TRIGGER: now also IC5.2; no longer IC4.2
- net U_CAM2_TRIGGER: now also IC4.2; no longer IC2.2
- net U_LICK_PORT_1: now also IC2.4; no longer IC6.4
- net U_LICK_PORT_2: now also IC9.4; no longer IC5.4
Routing:
- net +3V3_U: track 108.3 -> 101.3 mm
- net +3V3: track 200.1 -> 206.2 mm
- net PDI_DATA: track 15.3 -> 10.3 mm
- net PDI_CLK: track 12.1 -> 16.9 mm
- net N$14: track 6.87 -> 9.31 mm
- net +5V: track 100.0 -> 98.4 mm
- net N$5: track 10.6 -> 12.2 mm
- net USBDM: track 10.4 -> 9.16 mm
- net USBDP: track 8.44 -> 7.30 mm
- net U_CAM2_TRIGGER: track 38.0 -> 39.1 mm
- net N$8: track 6.33 -> 5.43 mm
- net N$4: track 6.78 -> 5.99 mm
- net GND: vias 96 -> 99
- added copper zone on layer 1, net N$103
- added copper zone on layer 15, net N$58
- added copper zone on layer 2, net N$61
- removed copper zone on layer 2, net N$58
- removed copper zone on layer 15, net N$61
Other:
- board text added: "v.1.1"
- board text removed: "v1.0"
