File: Hardware/PCB/VestibularH1.sch (EAGLE design)
At the start: 67 parts, among them IC1 FT232RL, IC2 SN74LVC1G125DBVT, IC3 LP5907MFX-3.3, IC4 SN74LVC1G125DBVT, IC5 SN74LVC1G125DBVT, IC6 SN74LVC1G125DBVT, IC7 USBLC6-2SC6, IC8 ATXMEGA32A4U, T1 DMG1012UW, T2 DMG1012UW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

Commit message: Replaced files with version 1.1.
Parts:
- removed IC6: SN74LVC1G125DBVT, VestibularVR H1-module v1.0:74LVC1G07DBV
- added IC9: M74VHC1GT126DT1G, VestibularVR H1-module v1.0:M74VHC1GT126DT1G
- C10: device rcl:C-EUC0603K -> rcl:C-EUC0603
- IC2, IC4, IC5: value SN74LVC1G125DBVT -> M74VHC1GT126DT1G; device VestibularVR H1-module v1.0:74LVC1G07DBV -> VestibularVR H1-module v1.0:M74VHC1GT126DT1G; DIGIKEY_PN (none) -> M74VHC1GT126DT1GOSDKR-ND; MPN SN74LVC1G125DBVT -> M74VHC1GT126DT1G; OEPS OEPS080029 -> OEPS080017
- X1: MPN (none) -> 2x5 header
- renumbered REWARD_VALVES to VALVES
Connections:
- net +3V3: now also IC2.OE, IC2.VCC, IC9.OE, IC9.VCC; no longer IC5.VCC, IC6.VCC
- net +3V3_U: now also SV2.2; no longer SV2.6
- net GND: now also IC9.GND, SV2.6; no longer IC6.GND, SV2.2
- net LICK_PORT_1: now also IC2.A; no longer IC6.A
- net LICK_PORT_2: now also IC9.A; no longer IC5.A
- net N$14: now also IC4.OE, IC4.VCC; no longer IC2.VCC
- net N$4: now also IC4.Y; no longer IC2.Y
- net N$5: now also IC5.OE, IC5.VCC; no longer IC4.VCC
- net N$8: now also IC5.Y; no longer IC4.Y
- net PDI_CLK: now also SV2.5; no longer SV2.1
- net PDI_DATA: now also SV2.1; no longer SV2.5
- net USBDM: now also IC7.IO2@0; no longer IC7.IO1@0
- net USBDP: now also IC7.IO1@0; no longer IC7.IO2@0
- net U_CAM1_TRIGGER: now also IC5.A; no longer IC4.A
- net U_CAM2_TRIGGER: now also IC4.A; no longer IC2.A
- net U_LICK_PORT_1: now also IC2.Y; no longer IC6.Y
- net U_LICK_PORT_2: now also IC9.Y; no longer IC5.Y
Other:
- note added: "Valves"
- note removed: "- to review IC2, IC4, IC5, IC6 part nb corrected: - was set as 74VHC1GT126DT1G - was changed to SN74LVC1G125DBVT - both parts have Enable pin; pin not drawn in symbol - new part SN74LVC1G125DBVT more available in suppliers - Enable pin of 74VHC1GT126DT1G active high; - Enable pin of new SN74LVC1G125DBVT active low; > more safe; independent of voltage supply used - part number corrected - OEPS cod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"
- note removed: "-to review USBDP & USBDP pin switched!!!"
- note removed: "-to review pinout upside-down!!!"
- note removed: "DMG1012UW"
- note removed: "Lick port de OC maior R PDown ~50k"
- note removed: "PAA5100JE Optical tracking - can be powered @ 3V3 or 5V - line outputs level will depend of power"
- note removed: "Reward Valves"
- note removed: "lick sensor @3V3 GP1A57HRJ00F photointerrupter - design from FED3"
- moved on the sheet: C13, C15, C16, R34, SV2
